File: electronics/deltabot-heater-bed/deltabot-heater-bed.brd (EAGLE design)
At the start: 185.9 x 190.5 mm, 61 parts

Commit message: board is ready for rev a release.
Parts:
- H1, H2, H3: value MOUNT-HOLE3.2 -> MOUNT-HOLE3.0; device holes:3,2 -> holes:3,0
- moved LOGO1 0.53 mm to (-14.2, -11.2)
Other:
- board text added: "CAUTION: HOT SURFACE DO NOT TOUCH"
- board text added: "DELTABOT HEATED BED"
- board text added: "Revision A License: GPLv3 Copyright: 2013 Design by: Zach Hoeken github.com/Hoektronics/NiuB"
- board text removed: "GPLv3"
Changed lines of the file:
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@@
 <setting verticaltext="up"/>
 </settings>
-<grid distance="0.25" unitdist="mm" unit="mm" style="lines" multiple="1" display="yes" altdistance="0.025" altunitdist="inch" altunit="inch"/>
+<grid distance="5" unitdist="mm" unit="mm" style="lines" multiple="1" display="yes" altdistance="0.025" altunitdist="inch" altunit="inch"/>
 <layers>
 <layer number="1" name="Top" color="4" fill="1" visible="yes" active="yes"/>
@@
 <layer number="28" name="bValues" color="7" fill="1" visible="yes" active="yes"/>
 <layer number="29" name="tStop" color="7" fill="3" visible="yes" active="yes"/>
-<layer number="30" name="bStop" color="7" fill="6" visible="yes" active="yes"/>
-<layer number="31" name="tCream" color="7" fill="4" visible="yes" active="yes"/>
-<layer number="32" name="bCream" color="7" fill="5" visible="yes" active="yes"/>
-<layer number="33" name="tFinish" color="6" fill="3" visible="yes" active="yes"/>
-<layer number="34" name="bFinish" color="6" fill="6" visible="yes" active="yes"/>
-<layer number="35" name="tGlue" color="7" fill="4" visible="yes" active="yes"/>
-<layer number="36" name="bGlue" color="7" fill="5" visible="yes" active="yes"/>
-<layer number="37" name="tTest" color="7" fill="1" visible="yes" active="yes"/>
-<layer number="38" name="bTest" color="7" fill="1" visible="yes" active="yes"/>
-<layer number="39" name="tKeepout" color="4" fill="11" visible="yes" active="yes"/>
-<layer number="40" name="bKeepout" color="1" fill="11" visible="yes" active="yes"/>
-<layer number="41" name="tRestrict" color="4" fill="10" visible="yes" active="yes"/>
-<layer number="42" name="bRestrict" color="1" fill="10" visible="yes" active="yes"/>
+<layer number="30" name="bStop" color="7" fill="6" visible="no" active="yes"/>
+<layer number="31" name="tCream" color="7" fill="4" visible="no" active="yes"/>
+<layer number="32" name="bCream" color="7" fill="5" visible="no" active="yes"/>
+<layer number="33" name="tFinish" color="6" fill="3" visible="no" active="yes"/>
+<layer number="34" name="bFinish" color="6" fill="6" visible="no" active="yes"/>
+<layer number="35" name="tGlue" color="7" fill="4" visible="no" active="yes"/>
+<layer number="36" name="bGlue" color="7" fill="5" visible="no" active="yes"/>
+<layer number="37" name="tTest" color="7" fill="1" visible="no" active="yes"/>
+<layer number="38" name="bTest" color="7" fill="1" visible="no" active="yes"/>
+<layer number="39" name="tKeepout" color="4" fill="11" visible="no" active="yes"/>
+<layer number="40" name="bKeepout" color="1" fill="11" visible="no" active="yes"/>
+<layer number="41" name="tRestrict" color="4" fill="10" visible="no" active="yes"/>
+<layer number="42" name="bRestrict" color="1" fill="10" visible="no" active="yes"/>
 <layer number="43" name="vRestrict" color="2" fill="10" visible="yes" active="yes"/>
 <layer number="44" name="Drills" color="7" fill="1" visible="yes" active="yes"/>
@@
 <wire x1="20.54211875" y1="54.16291875" x2="40.54033125" y2="77.049759375" width="0.001" layer="49"/>
 <wire x1="28.55848125" y1="36.06146875" x2="57.11083125" y2="60.210140625" width="0.001" layer="49"/>
-<text x="-4.5" y="-12.5" size="1.778" layer="21" ratio="16">GPLv3</text>
+<text x="0" y="-50" size="10" layer="21" font="vector" ratio="16" align="center">DELTABOT
+HEATED BED</text>
+<text x="0" y="40" size="10" layer="21" font="vector" ratio="16" align="center">CAUTION:
+HOT SURFACE
+DO NOT TOUCH
+</text>
+<text x="0" y="-24" size="2.5" layer="21" font="vector" ratio="16" align="center">Revision A
+License: GPLv3
+Copyright: 2013
+Design by: Zach Hoeken
+github.com/Hoektronics/NiuB</text>
+<wire x1="-59.4639" y1="-10.0446" x2="-39.4639" y2="-10.0446" width="0.4064" layer="21"/>
+<wire x1="-39.4639" y1="-10.0446" x2="-49.4639" y2="7.9554" width="0.4064" layer="21"/>
+<wire x1="-49.4639" y1="7.9554" x2="-59.4639" y2="-10.0446" width="0.4064" layer="21"/>
+<wire x1="-47.4639" y1="-7.0446" x2="-47.4639" y2="-4.0446" width="0.4064" layer="21" curve="-90"/>
+<wire x1="-47.4639" y1="-4.0446" x2="-47.4639" y2="-0.0446" width="0.4064" layer="21" curve="90"/>
+<wire x1="-49.4639" y1="-7.0446" x2="-49.4639" y2="-4.0446" width="0.4064" layer="21" curve="-90"/>
+<wire x1="-49.4639" y1="-4.0446" x2="-49.4639" y2="-0.0446" width="0.4064" layer="21" curve="90"/>
+<wire x1="-51.4639" y1="-7.0446" x2="-51.4639" y2="-4.0446" width="0.4064" layer="21" curve="-90"/>
+<wire x1="-51.4639" y1="-4.0446" x2="-51.4639" y2="-0.0446" width="0.4064" layer="21" curve="90"/>
+<wire x1="-45.4639" y1="-8.0446" x2="-53.4639" y2="-8.0446" width="0.4064" layer="21"/>
+<wire x1="40.5361" y1="-10.0446" x2="60.5361" y2="-10.0446" width="0.4064" layer="21"/>
+<wire x1="60.5361" y1="-10.0446" x2="50.5361" y2="7.9554" width="0.4064" layer="21"/>
+<wire x1="50.5361" y1="7.9554" x2="40.5361" y2="-10.0446" width="0.4064" layer="21"/>
+<wire x1="52.5361" y1="-7.0446" x2="52.5361" y2="-4.0446" width="0.4064" layer="21" curve="-90"/>
+<wire x1="52.5361" y1="-4.0446" x2="52.5361" y2="-0.0446" width="0.4064" layer="21" curve="90"/>
+<wire x1="50.5361" y1="-7.0446" x2="50.5361" y2="-4.0446" width="0.4064" layer="21" curve="-90"/>
+<wire x1="50.5361" y1="-4.0446" x2="50.5361" y2="-0.0446" width="0.4064" layer="21" curve="90"/>
+<wire x1="48.5361" y1="-7.0446" x2="48.5361" y2="-4.0446" width="0.4064" layer="21" curve="-90"/>
+<wire x1="48.5361" y1="-4.0446" x2="48.5361" y2="-0.0446" width="0.4064" layer="21" curve="90"/>
+<wire x1="54.5361" y1="-8.0446" x2="46.5361" y2="-8.0446" width="0.4064" layer="21"/>
 </plain>
 <attributes>
@@
 </class>
 </classes>
-<designrules name="hoektronics">
+<designrules name="hoektronics *">
 <description language="en">&lt;b&gt;EAGLE Design Rules&lt;/b&gt;
 &lt;p&gt;
@@
 <param name="mlMinCreamFrame" value="4mil"/>
 <param name="mlMaxCreamFrame" value="4mil"/>
-<param name="mlViaStopLimit" value="25mil"/>
+<param name="mlViaStopLimit" value="100mil"/>
 <param name="srRoundness" value="0"/>
 <param name="srMinRoundness" value="0mil"/>
@@
 </autorouter>
 <elements>
-<element name="H1" library="holes" package="3,2" value="MOUNT-HOLE3.2" x="86.602534375" y="-49.999996875" rot="R330"/>
-<element name="H2" library="holes" package="3,2" value="MOUNT-HOLE3.2" x="-86.6025375" y="-49.999996875" rot="R210"/>
-<element name="H3" library="holes" package="3,2" value="MOUNT-HOLE3.2" x="0" y="100" rot="R90"/>
+<element name="H1" library="holes" package="3,0" value="MOUNT-HOLE3.0" x="86.602534375" y="-49.999996875" rot="R330"/>
+<element name="H2" library="holes" package="3,0" value="MOUNT-HOLE3.0" x="-86.6025375" y="-49.999996875" rot="R210"/>
+<element name="H3" library="holes" package="3,0" value="MOUNT-HOLE3.0" x="0" y="100" rot="R90"/>
 <element name="S1" library="SparkFun-Electromechanical" package="TACTILE_SWITCH_SMD" value="" x="77.942284375" y="-45" rot="R240">
 <attribute name="PROD_ID" value="SWCH-08247" x="77.942284375" y="-45" size="1.778" layer="27" rot="R240" display="off"/>
@@
 <element name="LED23" library="Hoektronics" package="0805-LED" value="" x="71.28169375" y="39.86566875" rot="MR330"/>
 <element name="R27" library="Hoektronics" package="0805-RC" value="" x="70.28169375" y="41.597721875" rot="MR330"/>
-<element name="SJ1" library="SparkFun-Passives" package="SJ_2S" value="SOLDERJUMPERNC" x="11" y="94.75" rot="MR90"/>
-<element name="SJ2" library="SparkFun-Passives" package="SJ_2S" value="SOLDERJUMPERNC" x="5" y="94.75" rot="MR90"/>
-<element name="LOGO1" library="ohw-logo" package="OSHW_FILLX1000_NOTEXT" value="OSHW_LOGO_FILLX1000-NT" x="-14.75" y="-11.25"/>
+<element name="SJ1" library="SparkFun-Passives" package="SJ_2S" value="SOLDERJUMPERNC" x="11" y="94.75" smashed="yes" rot="MR90">
+<attribute name="NAME" x="12.27" y="93.8002" size="0.4064" layer="26" rot="MR90"/>
+</element>
+<element name="SJ2" library="SparkFun-Passives" package="SJ_2S" value="SOLDERJUMPERNC" x="5" y="94.75" smashed="yes" rot="MR90">
+<attribute name="NAME" x="6.27" y="93.8002" size="0.4064" layer="26" rot="MR90"/>
+</element>
+<element name="LOGO1" library="ohw-logo" package="OSHW_FILLX1000_NOTEXT" value="OSHW_LOGO_FILLX1000-NT" x="-14.224" y="-11.25"/>
 </elements>
 <signals>
@@
 </board>
 </drawing>
+<compatibility>
+<note version="6.3" minversion="6.2.2" severity="warning">
+Since Version 6.2.2 text objects can contain more than one line,
+which will not be processed correctly with this version.
+</note>
+</compatibility>
 </eagle>
