File: electronics/extruder-flex-heater/extruder-flex-heater.sch (EAGLE design)
At the start: 4 parts

Commit message: heater boards ready for release.
Parts:
- R1: value (none) -> 1k
Other:
- note added: "Extruder Flexible PCB Heater Rev A"
- note added: "HEATER COIL"
- note added: "LED"
- note added: "Notes: * Designed for 12V operation * Flexible polyimide circuit, single layer * 1/2 oz copper * Calculations: http://goo.gl/0InPi * License: GPLv3 * Copyright 2013 Hoektronics * Source: https://github.com/Hoektronics/NiuB"
- moved on the sheet: +, -, LED1, R1
Changed lines of the file:
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@@
 <layers>
 <layer number="1" name="Top" color="4" fill="1" visible="no" active="no"/>
+<layer number="2" name="Route2" color="1" fill="3" visible="no" active="no"/>
+<layer number="3" name="Route3" color="4" fill="3" visible="no" active="no"/>
+<layer number="4" name="Route4" color="1" fill="4" visible="no" active="no"/>
+<layer number="5" name="Route5" color="4" fill="4" visible="no" active="no"/>
+<layer number="6" name="Route6" color="1" fill="8" visible="no" active="no"/>
+<layer number="7" name="Route7" color="4" fill="8" visible="no" active="no"/>
+<layer number="8" name="Route8" color="1" fill="2" visible="no" active="no"/>
+<layer number="9" name="Route9" color="4" fill="2" visible="no" active="no"/>
+<layer number="10" name="Route10" color="1" fill="7" visible="no" active="no"/>
+<layer number="11" name="Route11" color="4" fill="7" visible="no" active="no"/>
+<layer number="12" name="Route12" color="1" fill="5" visible="no" active="no"/>
+<layer number="13" name="Route13" color="4" fill="5" visible="no" active="no"/>
+<layer number="14" name="Route14" color="1" fill="6" visible="no" active="no"/>
+<layer number="15" name="Route15" color="4" fill="6" visible="no" active="no"/>
 <layer number="16" name="Bottom" color="1" fill="1" visible="no" active="no"/>
 <layer number="17" name="Pads" color="2" fill="1" visible="no" active="no"/>
@@
 <part name="+" library="wirepad" deviceset="SMD2" device=""/>
 <part name="LED1" library="Hoektronics" deviceset="LED" device="0805"/>
-<part name="R1" library="Hoektronics" deviceset="RESISTOR" device="0805"/>
+<part name="R1" library="Hoektronics" deviceset="RESISTOR" device="0805" value="1k"/>
+<part name="FRAME1" library="frames" deviceset="A4L-LOC" device=""/>
 </parts>
 <sheets>
 <sheet>
 <plain>
+<text x="78.74" y="101.6" size="1.778" layer="91">HEATER COIL</text>
+<text x="40.64" y="101.6" size="1.778" layer="91">LED</text>
+<text x="38.1" y="91.44" size="2.54" layer="91" align="top-left">Notes:
+* Designed for 12V operation
+* Flexible polyimide circuit, single layer
+* 1/2 oz copper
+* Calculations: http://goo.gl/0InPi
+* License: GPLv3
+* Copyright 2013 Hoektronics
+* Source: https://github.com/Hoektronics/NiuB</text>
+<text x="40.64" y="114.3" size="5.08" layer="91">Extruder Flexible PCB Heater Rev A</text>
 </plain>
 <instances>
-<instance part="-" gate="1" x="10.16" y="12.7"/>
-<instance part="+" gate="1" x="10.16" y="20.32"/>
-<instance part="LED1" gate="G$1" x="5.08" y="20.32" rot="R270"/>
-<instance part="R1" gate="G$1" x="2.54" y="12.7"/>
+<instance part="-" gate="1" x="63.5" y="99.06"/>
+<instance part="+" gate="1" x="63.5" y="106.68"/>
+<instance part="LED1" gate="G$1" x="58.42" y="106.68" rot="R270"/>
+<instance part="R1" gate="G$1" x="55.88" y="99.06"/>
+<instance part="FRAME1" gate="G$1" x="0" y="0"/>
 </instances>
 <busses>
@@
 <segment>
 <pinref part="-" gate="1" pin="P"/>
-<wire x1="12.7" y1="12.7" x2="22.86" y2="12.7" width="0.1524" layer="91"/>
-<wire x1="22.86" y1="12.7" x2="22.86" y2="20.32" width="0.1524" layer="91"/>
+<wire x1="66.04" y1="99.06" x2="76.2" y2="99.06" width="0.1524" layer="91"/>
+<wire x1="76.2" y1="99.06" x2="76.2" y2="106.68" width="0.1524" layer="91"/>
 <pinref part="+" gate="1" pin="P"/>
-<wire x1="22.86" y1="20.32" x2="12.7" y2="20.32" width="0.1524" layer="91"/>
+<wire x1="76.2" y1="106.68" x2="66.04" y2="106.68" width="0.1524" layer="91"/>
 <pinref part="LED1" gate="G$1" pin="A"/>
-<wire x1="12.7" y1="20.32" x2="7.62" y2="20.32" width="0.1524" layer="91"/>
-<junction x="12.7" y="20.32"/>
+<wire x1="66.04" y1="106.68" x2="60.96" y2="106.68" width="0.1524" layer="91"/>
+<junction x="66.04" y="106.68"/>
 <pinref part="R1" gate="G$1" pin="2"/>
-<wire x1="12.7" y1="12.7" x2="7.62" y2="12.7" width="0.1524" layer="91"/>
-<junction x="12.7" y="12.7"/>
+<wire x1="66.04" y1="99.06" x2="60.96" y2="99.06" width="0.1524" layer="91"/>
+<junction x="66.04" y="99.06"/>
 </segment>
 </net>
@@
 <pinref part="LED1" gate="G$1" pin="C"/>
 <pinref part="R1" gate="G$1" pin="1"/>
-<wire x1="-5.08" y1="12.7" x2="-2.54" y2="12.7" width="0.1524" layer="91"/>
-<wire x1="0" y1="20.32" x2="-5.08" y2="20.32" width="0.1524" layer="91"/>
-<wire x1="-5.08" y1="20.32" x2="-5.08" y2="12.7" width="0.1524" layer="91"/>
+<wire x1="48.26" y1="99.06" x2="50.8" y2="99.06" width="0.1524" layer="91"/>
+<wire x1="53.34" y1="106.68" x2="48.26" y2="106.68" width="0.1524" layer="91"/>
+<wire x1="48.26" y1="106.68" x2="48.26" y2="99.06" width="0.1524" layer="91"/>
 </segment>
 </net>
@@
 </schematic>
 </drawing>
+<compatibility>
+<note version="6.3" minversion="6.2.2" severity="warning">
+Since Version 6.2.2 text objects can contain more than one line,
+which will not be processed correctly with this version.
+</note>
+</compatibility>
 </eagle>
