File: electronics/extruder board/extruder board -- placement 2.sch (EAGLE design)
At the start: 22 parts, among them IC1 MAX6675, IC2 MAX6675, J1 Main THERMO, J2 AUX THERMO, J3 Main Heater, J4 Secondary HEATER, X1 22-23-2041, X2 Right Fan, X3 Left Fan, X4 Extruder Fan

Commit message: Revert "Updated extruder board V1.1"
This reverts commit 2d423195ed33dd4a98d803fb0bad6f27ea0b4d36.
Parts:
- removed C3, C4: 0.1uF, rcl:C-USC0603
- removed J1: Main THERMO, 555 delay toggle switch:CON-AMP_MTA02-156
- removed J2: AUX THERMO, 555 delay toggle switch:CON-AMP_MTA02-156
- removed J3: Main Heater, 555 delay toggle switch:CON-AMP_MTA02-156
- removed J4: Secondary HEATER, 555 delay toggle switch:CON-AMP_MTA02-156
- removed X1: 22-23-2041, con-molex:22-23-2041
- removed X2: Right Fan, con-molex:22-23-2021
- removed X3: Left Fan, con-molex:22-23-2021
- removed X4: Extruder Fan, con-molex:22-23-2021
- added AUX_THERMO, MAIN_HEATER, MAIN_THERMO, SECOND_HEATER: M023.5MM_LOCK, SparkFun-Connectors:M023.5MM_LOCK
- added EXTRUDER_FAN: M02POLAR_LOCK, extruder board -- placement 2:M02POLAR_LOCK
- added LEFT_FAN, RIGHT_FAN: M02JST-PTH-2, extruder board -- placement 2:M02JST-PTH-2
- added MOTOR: (no value), extruder board -- placement 2:M04POLAR_LOCK
- AUX_HEATER: value AUX HEATER -> (none)
- C1, C2: value 0.1uF -> (none)
- HEATER: value HEATER -> (none)
- POWER: value POWER -> (none)
- R1, R2, R3: value 1K -> (none)
Connections:
- removed net HEATER_GND: AUX_HEATER.C, HEATER.C, J3.1, J4.1, U$3.P$2, U$3.P$3
- net +12V: now also EXTRUDER_FAN.2, U$1.P$6; no longer U$1.P$2, X2-2.S, X3-2.S, X4-2.S
- net AUX_HEATER: now also SECOND_HEATER.1; no longer J4.2
- net COOLING_FANS: now also LEFT_FAN.2, RIGHT_FAN.2, U$1.P$5; no longer U$1.P$12, X2-1.S, X3-1.S
- net CS2!: now also U$1.P$10; no longer U$1.P$11
- net DO: now also U$1.P$11; no longer U$1.P$3
- net GND: now also AUX_HEATER.C, EXTRUDER_FAN.1, HEATER.C, LEFT_FAN.1, MAIN_HEATER.2, RIGHT_FAN.1, SECOND_HEATER.2, U$3.P$2, U$3.P$3; no longer X4-1.S
- net HEATER: now also MAIN_HEATER.1; no longer J3.2
- net MOTOR_A+: now also MOTOR.1, U$1.P$1; no longer U$1.P$4, X1-4.S
- net MOTOR_A-: now also MOTOR.2, U$1.P$2; no longer U$1.P$6, X1-3.S
- net MOTOR_B+: now also MOTOR.3, U$1.P$3; no longer U$1.P$8, X1-2.S
- net MOTOR_B-: now also MOTOR.4, U$1.P$4; no longer U$1.P$10, X1-1.S
- net N$1: now also IC1.T+, MAIN_THERMO.2; no longer C4.1, IC2.T-, J2.1
- net N$2: now also MAIN_THERMO.1; no longer C3.1, J1.1
- net N$3: now also AUX_THERMO.2, IC2.T+; no longer C3.2, IC1.T+, J1.2
- net N$4: now also AUX_THERMO.1, IC2.T-; no longer C4.2, IC2.T+, J2.2
- net SCK: now also U$1.P$12; no longer U$1.P$5
- net VCC: now also U$1.P$8; no longer U$1.P$1
Other:
- moved on the sheet: C1, IC2

Commit message: extruder board rev1
Parts:
- removed AUX_THERMO, MAIN_HEATER, MAIN_THERMO, SECOND_HEATER: M023.5MM_LOCK, SparkFun-Connectors:M023.5MM_LOCK
- removed EXTRUDER_FAN: M02POLAR_LOCK, extruder board -- placement 2:M02POLAR_LOCK
- removed LEFT_FAN, RIGHT_FAN: M02JST-PTH-2, extruder board -- placement 2:M02JST-PTH-2
- removed MOTOR: (no value), extruder board -- placement 2:M04POLAR_LOCK
- added C3, C4: 0.1uF, rcl:C-USC0603
- added J1: Main THERMO, 555 delay toggle switch:CON-AMP_MTA02-156
- added J2: AUX THERMO, 555 delay toggle switch:CON-AMP_MTA02-156
- added J3: Main Heater, 555 delay toggle switch:CON-AMP_MTA02-156
- added J4: Secondary HEATER, 555 delay toggle switch:CON-AMP_MTA02-156
- added X1: 22-23-2041, con-molex:22-23-2041
- added X2: Right Fan, con-molex:22-23-2021
- added X3: Left Fan, con-molex:22-23-2021
- added X4: Extruder Fan, con-molex:22-23-2021
- AUX_HEATER: value (none) -> AUX HEATER
- C1, C2: value (none) -> 0.1uF
- HEATER: value (none) -> HEATER
- POWER: value (none) -> POWER
- R1, R2, R3: value (none) -> 1K
Connections:
- new net HEATER_GND: AUX_HEATER.C, HEATER.C, J3.1, J4.1, U$3.P$2, U$3.P$3
- net +12V: now also X4-2.S; no longer EXTRUDER_FAN.2
- net AUX_HEATER: now also J4.2; no longer SECOND_HEATER.1
- net COOLING_FANS: now also X2-2.S, X3-2.S; no longer LEFT_FAN.2, RIGHT_FAN.2
- net GND: now also X2-1.S, X3-1.S, X4-1.S; no longer AUX_HEATER.C, EXTRUDER_FAN.1, HEATER.C, LEFT_FAN.1, MAIN_HEATER.2, RIGHT_FAN.1, SECOND_HEATER.2, U$3.P$2, U$3.P$3
- net HEATER: now also J3.2; no longer MAIN_HEATER.1
- net MOTOR_A+: now also X1-4.S; no longer MOTOR.1
- net MOTOR_A-: now also X1-3.S; no longer MOTOR.2
- net MOTOR_B+: now also X1-2.S; no longer MOTOR.3
- net MOTOR_B-: now also X1-1.S; no longer MOTOR.4
- net N$1: now also C4.1, IC2.T-, J2.1; no longer IC1.T+, MAIN_THERMO.2
- net N$2: now also C3.1, J1.1; no longer MAIN_THERMO.1
- net N$3: now also C3.2, IC1.T+, J1.2; no longer AUX_THERMO.2, IC2.T+
- net N$4: now also C4.2, IC2.T+, J2.2; no longer AUX_THERMO.1, IC2.T-
Other:
- moved on the sheet: C1, IC2
